File: main-board/main-board.kicad_sch (KiCad schematic)
At the start: 0 parts

Commit message: Add TSOP module
Parts:
- added C1: 0.1uF, symbol Device:C
- added R1: 1K, symbol Device:R
- added U1: TSOP382xx, OptoDevice:Vishay_MINICAST-3Pin, symbol Interface_Optical:TSOP382xx
- added U2: XIAO ESP32C3, XIAO_ESP32C3:xiao_esp32c3, symbol xiao_esp32c3:XIAO ESP32C3
Connections:
- new net: C1.1, R1.1, U1.3 (Vs)
- new net +3.3V: R1.2
- new net GNDS: C1.2, U1.2 (GND)
